File: proves_canted_turnstile/proves_canted_turnstile.kicad_sch (KiCad schematic)
At the start: 34 parts, among them J1 Conn_Coaxial, J10 WDT Disable Jumper, J11 DEBUG, J12 USB_C_Receptacle_USB2.0_16P, J3 Battery Charge Bypass, J6 FC Reset Jumper, J7 FC USB Bootselect Jumper, J8 USB_C_Receptacle_USB2.0_16P, J9 DF11-4DP-2DSA, U1 QBA-07+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

Commit message: implemented RF Switch
Parts:
- added J13: DF11-4DP-2DSA, Connector_Hirose:Hirose_DF11-4DP-2DSA_2x02_P2.00mm_Vertical, symbol Connector_Generic:Conn_02x02_Odd_Even
- added J2: Conn_Coaxial, Connector_Coaxial:MMCX_Molex_73415-1471_Vertical, symbol Connector:Conn_Coaxial
- added U4: PE4256, symbol pSEMI:PE4259
Connections:
- net +3V3: now also U4.6 (VDD/~{CTRL})
- net GND: now also J13.1 (Pin_1), J13.3 (Pin_3), J2.2 (Ext), U4.2 (GND)
- net UHF: now also U4.5 (RFC); no longer J1.1 (In)
- new net: J1.1 (In), U4.3 (RF2)
- new net: J2.1 (In), U4.1 (RF1)
- new net: J13.2 (Pin_2), J13.4 (Pin_4), U4.4 (CTRL)
Other:
- note added: "PROVES Radio"
- note added: "SATNOGS Comms"
- moved on the sheet: AE1, AE2, AE3, AE4, H1, H2, H3, H4, J1, R1, R2, R3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

Commit message: updated usb differential pair track widths
Parts:
- added Q1: Si7454DP, Package_SO:PowerPAK_SO-8_Single, symbol Transistor_FET:Si7450DP
- U4: footprint (none) -> Package_TO_SOT_SMD:SOT-363_SC-70-6
Connections:
- net +3V3: now also Q1.5 (D)
- net GND: now also J13.2 (Pin_2), J13.4 (Pin_4); no longer J13.1 (Pin_1), J13.3 (Pin_3)
- net PROVES_PORT: now reaches J1.1 (In), U4.3 (RF2)
- net SATNOGS_PORT: now reaches J2.1 (In), U4.1 (RF1)
- new net RF_PORT_CTRL: J13.1 (Pin_1), J13.3 (Pin_3), Q1.1 (S), Q1.2 (S), Q1.3 (S), Q1.4 (G), U4.4 (CTRL)
Other:
- moved on the sheet: H1, H2, H3, H4, J1

Commit message: fixed net labels
Connections:
- net RF_PORT_CTRL: no longer Q1.1 (S), Q1.2 (S), Q1.3 (S), U4.4 (CTRL)
- new net CTRL: Q1.1 (S), Q1.2 (S), Q1.3 (S), U4.4 (CTRL)
Changed lines of the file:
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@@
 		)
 	)
-	(label "RF_PORT_CTRL"
+	(label "CTRL"
 		(at 143.51 85.09 270)
 		(effects

Commit message: removed burnwire resistor and fixed up some traces
Parts:
- removed R4: R_Small_US, Resistor_THT:R_Axial_DIN0309_L9.0mm_D3.2mm_P12.70mm_Horizontal, symbol Device:R_Small_US
- U4: footprint Package_TO_SOT_SMD:SOT-363_SC-70-6 -> Package_TO_SOT_SMD:SOT-363_SC-70-6_Handsoldering
Other:
- note removed: "Burnwire"
Changed lines of the file:
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@@
 		)
 	)
-	(text "Burnwire"
-		(exclude_from_sim no)
-		(at 342.9 175.006 0)
-		(effects
-			(font
-				(size 1.27 1.27)
-			)
-		)
-	)
 	(junction
 		(at 134.62 114.3)
@@
 	(wire
 		(pts
-			(xy 361.95 185.42) (xy 361.95 189.23)
-		)
-		(stroke
-			(width 0)
-			(type default)
-		)
-	)
-	(wire
-		(pts
 			(xy 68.58 220.98) (xy 68.58 218.44)
 		)
@@
 	(wire
 		(pts
-			(xy 359.41 185.42) (xy 361.95 185.42)
-		)
-		(stroke
-			(width 0)
-			(type default)
-		)
-	)
-	(wire
-		(pts
 			(xy 208.28 217.17) (xy 208.28 220.98)
 		)
@@
 	(wire
 		(pts
-			(xy 334.01 185.42) (xy 354.33 185.42)
-		)
-		(stroke
-			(width 0)
-			(type default)
-		)
-	)
-	(wire
-		(pts
 			(xy 218.44 115.57) (xy 213.36 115.57)
 		)
@@
 		)
 	)
-	(global_label "BURN"
-		(shape input)
-		(at 334.01 185.42 180)
-		(fields_autoplaced yes)
-		(effects
-			(font
-				(size 1.27 1.27)
-			)
-			(justify right)
-		)
-		(property "Intersheetrefs" "${INTERSHEET_REFS}"
-			(at 325.8238 185.42 0)
-			(effects
-				(font
-					(size 1.27 1.27)
-				)
-				(justify right)
-				(hide yes)
-			)
-		)
-	)
 	(global_label "FC_USBBOOT"
 		(shape output)
@@
 			)
 		)
-		(property "Footprint" "Package_TO_SOT_SMD:SOT-363_SC-70-6"
+		(property "Footprint" "Package_TO_SOT_SMD:SOT-363_SC-70-6_Handsoldering"
 			(at 120.65 83.82 0)
 			(effects
@@
 	)
 	(symbol
-		(lib_id "Device:R_Small_US")
-		(at 356.87 185.42 90)
-		(unit 1)
-		(exclude_from_sim no)
-		(in_bom yes)
-		(on_board yes)
-		(dnp no)
-		(fields_autoplaced yes)
-		(property "Reference" "R4"
-			(at 356.87 179.07 90)
-			(effects
-				(font
-					(size 1.27 1.27)
-				)
-			)
-		)
-		(property "Value" "R_Small_US"
-			(at 356.87 181.61 90)
-			(effects
-				(font
-					(size 1.27 1.27)
-				)
-			)
-		)
-		(property "Footprint" "Resistor_THT:R_Axial_DIN0309_L9.0mm_D3.2mm_P12.70mm_Horizontal"
-			(at 356.87 185.42 0)
-			(effects
-				(font
-					(size 1.27 1.27)
-				)
-				(hide yes)
-			)
-		)
-		(property "Datasheet" "~"
-			(at 356.87 185.42 0)
-			(effects
-				(font
-					(size 1.27 1.27)
-				)
-				(hide yes)
-			)
-		)
-		(property "Description" "Resistor, small US symbol"
-			(at 356.87 185.42 0)
-			(effects
-				(font
-					(size 1.27 1.27)
-				)
-				(hide yes)
-			)
-		)
-		(pin "1"
-		)
-		(pin "2"
-		)
-		(instances
-			(project ""
-				(path "/b0a1b345-df47-405c-b751-07790b55dab3"
-					(reference "R4")
-					(unit 1)
-				)
-			)
-		)
-	)
-	(symbol
 		(lib_id "Mechanical:MountingHole")
 		(at 72.39 135.89 0)
@@
 					(unit 1)
 				)
-			)
-		)
-	)
-	(symbol
-		(lib_id "power:GND")
-		(at 361.95 189.23 0)
-		(unit 1)
-		(exclude_from_sim no)
-		(in_bom yes)
-		(on_board yes)
-		(dnp no)
-		(fields_autoplaced yes)
-		(property "Reference" "#PWR01"
-			(at 361.95 195.58 0)
-			(effects
-				(font
-					(size 1.27 1.27)
-				)
-				(hide yes)
-			)
-		)
-		(property "Value" "GND"
-			(at 361.95 194.31 0)
-			(effects
-				(font
-					(size 1.27 1.27)
-				)
-			)
-		)
-		(property "Footprint" ""
-			(at 361.95 189.23 0)
-			(effects
-				(font
-					(size 1.27 1.27)
-				)
-				(hide yes)
-			)
-		)
-		(property "Datasheet" ""
-			(at 361.95 189.23 0)
-			(effects
-				(font
-					(size 1.27 1.27)
-				)
-				(hide yes)
-			)
-		)
-		(property "Description" "Power symbol creates a global label with name \"GND\" , ground"
-			(at 361.95 189.23 0)
-			(effects
-				(font
-					(size 1.27 1.27)
-				)
-				(hide yes)
-			)
-		)
-		(pin "1"
-		)
-		(instances
-			(project ""
-				(path "/b0a1b345-df47-405c-b751-07790b55dab3"
-					(reference "#PWR01")
-					(unit 1)
-				)

Commit message: gerber files and minor modifications
Parts:
- U4: value PE4256 -> PE4259
Changed lines of the file:
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@@
 			)
 		)
-		(property "Value" "PE4256"
+		(property "Value" "PE4259"
 			(at 128.905 68.58 0)
 			(effects
