File: antenna_top_cap_v2c/antenna_top_cap_v2c.kicad_pcb (KiCad board)
At the start: 4 copper layers, 100 x 100 mm, 55 parts, among them J1 DEBUG, J10 WDT Disable Jumper, J11 DF11-4DP-2DSA, J12 USB_C_Receptacle_USB2.0_16P, J13 DNP, J2 Battery Charge Bypass, J3 FC Reset Jumper, J4 FC USB Bootselect Jumper, J8 USB_C_Receptacle_USB2.0_16P, J9 DF11-4DP-2DSA, Q2 CSD17576Q5B, U3 VEML6031X00, U4 TMP112xxDRL, U6 TCA4311ADGKR

Commit message: Removed Legacy RBF Holes
Parts:
- removed TP2, TP3, TP7: TestPoint, MountingHole:MountingHole_2.7mm_M2.5_Pad
Other:
- board text added: "3PySquared Antenna Board V2c Michael Pham | Nicole Maggard | Ernesto Montes"
- board text removed: "3PySquared Antenna Board V2b Michael Pham | Nicole Maggard | Ernesto Montes"
